File: KiCad/KiCad.kicad_sch (KiCad schematic)
At the start: 71 parts, among them J1 Barrel_Jack_Switch, J2 UC_CONN_01X02, J3 UC_CONN_01X02, J4 MOTOR-L, J5 MOTOR-R, J6 Conn_01x15_Socket, J7 Conn_01x15_Socket, Q1 BSH205, Q2 BSH205, Q3 BSH205, Q4 BSH205, Q5 BSH205, SW1 SW_SPST, SW2 UC_SW_Push, SW3 UC_SW_Push, U1 LM338T, U2 ZXBM5210-S, U3 ZXBM5210-S, U4 74HC595, U5 74HC595

Commit message: Finished Rev A schematic
Parts:
- removed SW2: UC_SW_Push, Button_Switch_THT:SW_PUSH_6mm_H5mm, symbol enel200_uc_kicad7:UC_SW_Push
- added C12: 10uF, Capacitor_THT:CP_Radial_D5.0mm_P2.00mm, symbol enel200_uc_kicad7:UC_CP
- added J10, J12: 3v3, Connector_PinHeader_2.54mm:PinHeader_1x02_P2.54mm_Vertical, symbol enel200_uc_kicad7:UC_CONN_01X02
- added J11, J13: 5v, Connector_PinHeader_2.54mm:PinHeader_1x02_P2.54mm_Vertical, symbol enel200_uc_kicad7:UC_CONN_01X02
- added J14, J15: ESP_PT, symbol Connector_Generic:Conn_01x15
- added J8: LEAF_L, Connector_PinHeader_2.54mm:PinHeader_1x02_P2.54mm_Vertical, symbol enel200_uc_kicad7:UC_CONN_01X02
- added J9: LEAF_R, Connector_PinHeader_2.54mm:PinHeader_1x02_P2.54mm_Vertical, symbol enel200_uc_kicad7:UC_CONN_01X02
- added R15, R16: 1k, Resistor_THT:R_Axial_DIN0207_L6.3mm_D2.5mm_P7.62mm_Horizontal, symbol enel200_uc_kicad7:UC_R
- added R17, R9: 3k3, Resistor_THT:R_Axial_DIN0207_L6.3mm_D2.5mm_P7.62mm_Horizontal, symbol enel200_uc_kicad7:UC_R
- added R7, R8: 10k, Resistor_THT:R_Axial_DIN0207_L6.3mm_D2.5mm_P7.62mm_Horizontal, symbol enel200_uc_kicad7:UC_R
- added SW5: BTN_B, Button_Switch_THT:SW_PUSH_6mm_H5mm, symbol enel200_uc_kicad7:UC_SW_Push
- added U6: LM1117T-3.3, Package_TO_SOT_THT:TO-220-3_Horizontal_TabDown, symbol Regulator_Linear:LM1117T-3.3
- D9: footprint (none) -> LED_SMD:LED_0603_1608Metric
- J2: value UC_CONN_01X02 -> PHOTORESISTOR_1
- J3: value UC_CONN_01X02 -> PHOTORESISTOR_2
- J6, J7: value Conn_01x15_Socket -> ESP
- SW3: value UC_SW_Push -> BTN_A
Connections:
- net +5V: now also J11.2 (P2), J13.2 (P2)
- net GND: now also J2.1 (P1), J3.1 (P1), U4.8 (GND), U5.8 (GND), C12.2, J10.1 (P1), J11.1 (P1), J12.1 (P1), J13.1 (P1), J14.1 (Pin_1), R17.2, R9.1, U6.1 (GND)
- net GPIO4: now also J14.10 (Pin_10)
- net GPIO5: now also J14.9 (Pin_9)
- net GPIO6: now also J14.8 (Pin_8)
- net GPIO7: now also J14.7 (Pin_7)
- net PWR_IN: now also U6.3 (VI)
- net VDD: no longer J6.14 (Pin_14)
- net at U5.14 (SER): now also U4.9 (QH')
- net +3V3: now reaches U5.16 (VCC)
- net +3V3: now also J6.3 (Pin_3), SW3.1, U4.16 (VCC), C12.1, J10.2 (P2), J12.2 (P2), J14.13 (Pin_13), J8.2 (P2), J9.2 (P2), SW5.1, U6.2 (VO)
- net GPIO10: now reaches U4.10 (~{SRCLR})
- net GPIO10: now also J7.7 (Pin_7), J15.9 (Pin_9)
- net GPIO9: now reaches U4.11 (SRCLK)
- net GPIO9: now also J6.12 (Pin_12), J14.4 (Pin_4)
- net GPIO8: now reaches U4.14 (SER)
- net GPIO8: now also J6.11 (Pin_11), J14.5 (Pin_5)
- net at J2.2 (P2): now also R7.2
- net at J3.2 (P2): now also R8.2
- net at J7.1 (Pin_1): now also J15.15 (Pin_15)
- net at J7.10 (Pin_10): now also J15.6 (Pin_6)
- net at J7.11 (Pin_11): now also J15.5 (Pin_5)
- net GPIO18: now reaches J7.12 (Pin_12)
- net GPIO18: now also J15.4 (Pin_4), R7.1
- net GPIO19: now reaches J7.13 (Pin_13)
- net GPIO19: now also J15.3 (Pin_3), R8.1
- net at J7.14 (Pin_14): now also J15.2 (Pin_2)
- net at J7.15 (Pin_15): now also J15.1 (Pin_1)
- net GPIO0: now reaches J7.2 (Pin_2)
- net GPIO0: now also J15.14 (Pin_14), R15.1
- net GPIO1: now reaches J7.3 (Pin_3)
- net GPIO1: now also J15.13 (Pin_13), R16.1
- net at J7.4 (Pin_4): now also J15.12 (Pin_12)
- net at J7.5 (Pin_5): now also J15.11 (Pin_11)
- net at J7.6 (Pin_6): now also J15.10 (Pin_10)
- net at J7.8 (Pin_8): now also J15.8 (Pin_8)
- net at J7.9 (Pin_9): now also J15.7 (Pin_7)
- net at SW3.2: now also J8.1 (P1), R15.2, R9.2
- net at J6.1 (Pin_1): now also J14.15 (Pin_15)
- net at J6.10 (Pin_10): now also J14.6 (Pin_6)
- net at J6.13 (Pin_13): now also J14.3 (Pin_3)
- net at J6.2 (Pin_2): now also J14.14 (Pin_14)
- net at J6.4 (Pin_4): now also J14.12 (Pin_12)
- net at J6.5 (Pin_5): now also J14.11 (Pin_11)
- new net: J9.1 (P1), R16.2, R17.1, SW5.2
- new net: J14.2 (Pin_2), J6.14 (Pin_14)
Other:
- note added: "3v3 1A MAX."
- note added: "Breadboard Power Headers"
- note added: "Button Inputs"
- note added: "Connect to left and right power rails of the breadboard"
- note added: "Logic Linear Regulator"
- note added: "Motor Linear Regulator"
- note added: "PCB Power Headers"
- note added: "Pull-down resistors and guard resistors"
- note added: "Shift Registers"
- note added: "Two additional headers on top side of PCB"
- note removed: "Linear Regulator"
- note removed: "buttons leaf switch pullup / guard / connectors breadboard mounts"
- moved on the sheet: C1, C10, C2, C3, C4, C5, C6, C7, C8, C9, D1, D10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

Commit message: Added NC markers, title and date
Connections:
- no-connect marks 0 -> 13
Other:
- company: (none) -> C. Varney, A. Walker, K. Jones
- title: (none) -> ESP32 Breadboard Robot Breakout
Changed lines of the file:
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@@
 (kicad_sch (version 20230121) (generator eeschema)
   (paper "A3")
+  (title_block
+    (title "ESP32 Breadboard Robot Breakout")
+    (date "2024-09-21")
+    (rev "A")
+    (company "C. Varney, A. Walker, K. Jones")
+  )
   (junction (at 283.845 35.56) (diameter 0) (color 0 0 0 0)
   )
@@
   (junction (at 158.75 137.795) (diameter 0) (color 0 0 0 0)
   )
+  (no_connect (at 154.305 186.055))
+  (no_connect (at 90.17 182.88))
+  (no_connect (at 110.49 185.42))
+  (no_connect (at 110.49 182.88))
+  (no_connect (at 133.985 175.895))
+  (no_connect (at 133.985 180.975))
+  (no_connect (at 90.17 180.34))
+  (no_connect (at 133.985 173.355))
+  (no_connect (at 133.985 183.515))
+  (no_connect (at 154.305 183.515))
+  (no_connect (at 110.49 180.34))
+  (no_connect (at 154.305 180.975))
+  (no_connect (at 154.305 191.135))
   (wire (pts (xy 171.45 78.74) (xy 171.45 74.295))
     (stroke (width 0) (type default))

Commit message: PCB Revision A Created
Parts:
- removed J10: 3v3, Connector_PinHeader_2.54mm:PinHeader_1x02_P2.54mm_Vertical, symbol enel200_uc_kicad7:UC_CONN_01X02
- removed J11: 5v, Connector_PinHeader_2.54mm:PinHeader_1x02_P2.54mm_Vertical, symbol enel200_uc_kicad7:UC_CONN_01X02
- removed SW1: SW_SPST, symbol Switch:SW_SPST
- added R18: 330, Resistor_THT:R_Axial_DIN0207_L6.3mm_D2.5mm_P2.54mm_Vertical, symbol enel200_uc_kicad7:UC_R
- added SW2: SW_SPDT, Button_Switch_THT:SW_Slide-03_Wuerth-WS-SLTV_10x2.5x6.4_P2.54mm, symbol Switch:SW_SPDT
- D10, D11, D12, D13, D14, D15, D16, D17, D18, D19, D20, D21, D22, D23, D24, D25, D26, D27, D28, D29, D30, D6, D7, D8: footprint (none) -> LED_SMD:LED_1206_3216Metric_Pad1.42x1.75mm_HandSolder
- D5: footprint (none) -> LED_THT:LED_D5.0mm
- D9: footprint LED_SMD:LED_0603_1608Metric -> LED_SMD:LED_1206_3216Metric_Pad1.42x1.75mm_HandSolder
- J12: value 3v3 -> 3V3
- J13: value 5v -> 3V3
- J14, J15, J6, J7: footprint (none) -> Connector_PinHeader_2.54mm:PinHeader_1x15_P2.54mm_Vertical
- Q1, Q2, Q3, Q4, Q5: footprint Package_TO_SOT_THT:TO-92_Wide -> Package_TO_SOT_SMD:SOT-23-3
- R1, R10, R11, R12, R13, R14, R15, R16, R17, R2, R3, R4, R5, R6, R7, R8, R9: footprint Resistor_THT:R_Axial_DIN0207_L6.3mm_D2.5mm_P7.62mm_Horizontal -> Resistor_THT:R_Axial_DIN0207_L6.3mm_D2.5mm_P2.54mm_Vertical
- U4, U5: footprint (none) -> Package_SO:SOIC-16_4.55x10.3mm_P1.27mm
Connections:
- net +3V3: now also J13.2 (P2), J14.3 (Pin_3), J2.2 (P2), J3.2 (P2), Q1.3 (S), Q2.3 (S), Q3.3 (S), Q4.3 (S), Q5.3 (S); no longer J14.13 (Pin_13)
- net +5V: no longer J13.2 (P2)
- net COL1: now also Q1.2 (G), U4.1 (QB); no longer R10.1, U5.15 (QA)
- net COL2: now also Q2.2 (G), U4.2 (QC); no longer R11.1, U5.1 (QB)
- net COL3: now also Q3.2 (G), U4.3 (QD); no longer R12.1, U5.2 (QC)
- net COL4: now also Q4.2 (G), U4.4 (QE); no longer R13.1, U5.3 (QD)
- net COL5: now also Q5.2 (G), U4.5 (QF); no longer R14.1, U5.4 (QE)
- net GND: now also J14.15 (Pin_15), R7.2, R8.2; no longer J14.1 (Pin_1), J2.1 (P1), J3.1 (P1)
- net GPIO0: now also J15.2 (Pin_2), J2.1 (P1), R7.1; no longer J15.14 (Pin_14), R15.1
- net GPIO1: now also J15.3 (Pin_3); no longer J15.13 (Pin_13)
- net GPIO10: now also J15.7 (Pin_7), R6.1, U3.5 (REV); no longer J15.9 (Pin_9), U4.10 (~{SRCLR})
- net GPIO18: now also J15.12 (Pin_12), R4.1, U3.4 (FWD); no longer J15.4 (Pin_4), R7.1
- net GPIO19: now also J15.13 (Pin_13), U4.10 (~{SRCLR}); no longer J15.3 (Pin_3), R8.1
- net GPIO4: now also J14.6 (Pin_6), J3.1 (P1), R8.1; no longer J14.10 (Pin_10), R3.1, U2.4 (FWD)
- net GPIO5: now also J14.7 (Pin_7), R15.1; no longer J14.9 (Pin_9), R5.1, U2.5 (REV)
- net GPIO6: now also R3.1, U2.4 (FWD); no longer R4.1, U3.4 (FWD)
- net GPIO7: now also J14.9 (Pin_9), R5.1, U2.5 (REV); no longer J14.7 (Pin_7), R6.1, U3.5 (REV)
- net GPIO8: now also J14.11 (Pin_11); no longer J14.5 (Pin_5)
- net GPIO9: now also J14.12 (Pin_12); no longer J14.4 (Pin_4)
- net MOTOR-L1: now also C7.2, D2.1 (K), J4.1 (P1), U2.7 (OUT2); no longer C7.1, D1.1 (K), J4.2 (P2), U2.1 (OUT1)
- net MOTOR-L2: now also C7.1, D1.1 (K), J4.2 (P2), U2.1 (OUT1); no longer C7.2, D2.1 (K), J4.1 (P1), U2.7 (OUT2)
- net MOTOR-R1: now also C8.2, D4.1 (K), U3.7 (OUT2); no longer C8.1, D3.1 (K), U3.1 (OUT1)
- net MOTOR-R2: now also C8.1, D3.1 (K), U3.1 (OUT1); no longer C8.2, D4.1 (K), U3.7 (OUT2)
- net PWR_IN: now also R18.1, SW2.3 (C); no longer D5.2 (A)
- net ROW1: now also R10.1, U5.5 (QF); no longer Q1.2 (G), U4.15 (QA)
- net ROW2: now also R11.1, U5.4 (QE); no longer Q2.2 (G), U4.1 (QB)
- net ROW3: now also R12.1, U5.3 (QD); no longer Q3.2 (G), U4.2 (QC)
- net ROW4: now also R13.1, U5.2 (QC); no longer Q4.2 (G), U4.3 (QD)
- net ROW5: now also R14.1, U5.1 (QB); no longer Q5.2 (G), U4.4 (QE)
- net VDD: no longer Q1.3 (S), Q2.3 (S), Q3.3 (S), Q4.3 (S), Q5.3 (S)
- net at J6.5 (Pin_5): now also J14.5 (Pin_5); no longer J14.11 (Pin_11)
- net at J6.4 (Pin_4): now also J14.4 (Pin_4); no longer J14.12 (Pin_12)
- net at J14.14 (Pin_14): now also J6.14 (Pin_14); no longer J6.2 (Pin_2)
- net at J6.1 (Pin_1): now also J14.1 (Pin_1); no longer J14.15 (Pin_15)
- net at J14.2 (Pin_2): now also J6.2 (Pin_2); no longer J6.14 (Pin_14)
- net at J6.13 (Pin_13): now also J14.13 (Pin_13); no longer J14.3 (Pin_3)
- net at J6.10 (Pin_10): now also J14.10 (Pin_10); no longer J14.6 (Pin_6)
- net at J1.1: now also SW2.2 (B)
- net at J7.1 (Pin_1): now also J15.1 (Pin_1); no longer J15.15 (Pin_15)
- net at J7.10 (Pin_10): now also J15.10 (Pin_10); no longer J15.6 (Pin_6)
- net at J7.11 (Pin_11): now also J15.11 (Pin_11); no longer J15.5 (Pin_5)
- net at J7.14 (Pin_14): now also J15.14 (Pin_14); no longer J15.2 (Pin_2)
- net at J7.15 (Pin_15): now also J15.15 (Pin_15); no longer J15.1 (Pin_1)
- net at J7.4 (Pin_4): now also J15.4 (Pin_4); no longer J15.12 (Pin_12)
- net at J7.5 (Pin_5): now also J15.5 (Pin_5); no longer J15.11 (Pin_11)
- net at J7.6 (Pin_6): now also J15.6 (Pin_6); no longer J15.10 (Pin_10)
- net at J7.9 (Pin_9): now also J15.9 (Pin_9); no longer J15.7 (Pin_7)
- new net: D5.2 (A), R18.2
- no-connect marks 13 -> 14
Other:
- note removed: "Breadboard Power Headers"
- note removed: "Connect to left and right power rails of the breadboard"
- moved on the sheet: J14, J15, J2, J8, J9, R15, R16, R17, R9, SW3, SW5
