File: KiCad/KiCad.kicad_pcb (KiCad board)
At the start: 2 copper layers, 88.3 x 81.8 mm, 86 parts, among them J1 Barrel_Jack_Switch, J12 3V3, J13 3V3, J14 ESP_PT, J15 ESP_PT, J2 PHOTORESISTOR_1, J3 PHOTORESISTOR_2, J4 MOTOR-L, J5 MOTOR-R, J6 ESP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

Commit message: fixed connors clever commit
Parts:
- moved SW3 1.17 mm to (168.6, 110.2)
Routing:
- net +3V3: track 360.8 -> 364.4 mm
- net Net-(J8-P1): track 31.2 -> 28.1 mm
- net GPIO6: track 25.1 -> 27.7 mm
- net GPIO7: track 26.1 -> 28.5 mm
- net PWR_IN: track 39.2 -> 40.8 mm
