File: KiCad/ENEL200Group01.kicad_sch (KiCad schematic)
At the start: 86 parts, among them J1 Barrel_Jack_Switch, J12 3V3, J13 3V3, J14 ESP_PT, J15 ESP_PT, J2 PHOTORESISTOR_1, J3 PHOTORESISTOR_2, J4 MOTOR-L, J5 MOTOR-R, J6 ESP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

Commit message: final pcb rev
Parts:
- added C11, C13: 100nF, Capacitor_THT:C_Rect_L7.0mm_W2.5mm_P5.00mm, symbol enel200_uc_kicad7:UC_C
Connections:
- net +3V3: now also C11.1, C13.1
- net GND: now also C11.2, C13.2
